File: pcb/hall-effect.sch (KiCad schematic (older format))
At the start: 15 parts

Commit message: added usb interface, switching signal to boost circuits
Connections:
- new net: IC?.~, IC?.~ (x2)
Changed lines of the file:
@@
 $Descr A4 11693 8268
 encoding utf-8
-Sheet 3 4
+Sheet 3 5
 Title "Hall-effect sensor"
 Date ""
